File: schematics/hand sensor/EMG3.brd (EAGLE design)
At the start: 160 x 100 mm, 100 parts, among them IC1 INA118P, IC10 INA118P, IC11 OP275P, IC12 OP275P, IC2 OP275P, IC3 OP275P, IC4 INA118P, IC5 OP275P, IC6 OP275P, IC7 INA118P, IC8 OP275P, IC9 OP275P

Commit message: implement NN, dummy data, 3d hand
Parts:
- removed C10, C11, C17, C18, C24, C25: 220nF, rcl:C050-035X075
- removed C12, C19, C26: 33nF, rcl:C050-035X075
- removed C13, C20, C27: 22nF, rcl:C050-035X075
- removed C14, C21, C28: 100nF, rcl:C050-035X075
- removed C15, C16, C22, C23, C29, C30: 10nF, rcl:C050-035X075
- removed IC10, IC4, IC7: INA118P, burr-brown:DIL08
- removed IC11, IC12, IC5, IC6, IC8, IC9: OP275P, linear:DIL08
- removed R11, R25, R38, R51: 200, rcl:0207/7
- removed R15, R29, R42: 6.8k, rcl:0207/7
- removed R16, R21, R30, R34, R43, R47: 20k, rcl:0207/7
- removed R17, R26, R31, R39, R44, R52, RG1, RG2, RG3: 1K, rcl:0207/7
- removed R18, R32, R45: 100K, rcl:0207/7
- removed R20, R33, R46: 5.1k, rcl:0207/7
- removed R22, R27, R35, R40, R48: 51k, rcl:0207/7
- removed R23, R24, R36, R37, R49, R50: 10k, rcl:0207/7
- removed R28, R41, R9: 51K, rcl:0207/7
- added J1: AUDIO_JACK_3.5MM_PTH, SparkFun-Connectors:AUDIO-JACK
- C1, C2, C3, C4, C8, C9: device rcl:C050-035X075 -> rcl:C050-025X075
- R1, R10, R12, R13, R14, R19, R2, R3, R4, R6, R7, R8, RG: device rcl:0207/7 -> rcl:0207/12
- R5: value 51k -> (none); device rcl:0207/7 -> rcl:RTRIM64W
- moved R14 189.0 mm to (100.3, 92.7)
- moved R10 180.4 mm to (100.3, 87.6)
- moved R5 165.3 mm to (50.8, 92.7)
- moved C1 154.3 mm to (104.1, 64.8)
- moved C2 154.3 mm to (95.2, 64.8)
- moved C5 153.9 mm to (92.7, 72.4)
- moved C9 153.9 mm to (104.1, 72.4)
- moved IC1 150.6 mm to (101.6, 55.9)
- moved R8 149.4 mm to (69.8, 82.5)
- moved R2 145.0 mm to (100.3, 77.5)
- moved R6 144.6 mm to (100.3, 82.5)
- moved C6 142.7 mm to (64.8, 54.6)
- moved R3 140.2 mm to (85.1, 77.5)
- moved R7 139.8 mm to (85.1, 82.5)
- moved R19 130.1 mm to (85.1, 92.7)
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Connections:
- removed net N$18 (its old number): IC4.8, RG1.1
- removed net N$21: C10.1, IC4.6
- removed net N$22: C10.2, C11.1, R9.1
- removed net N$24: C11.2, IC5.5, R22.2
- removed net N$27: IC5.6, IC5.7, R15.2, R9.2
- removed net N$28: C12.2, R15.1, R16.2
- removed net N$29: C13.1, IC5.3, R16.1
- removed net N$30: C12.1, IC5.1, IC5.2, R20.2
- removed net N$31: IC6.2, R17.1, R18.2
- removed net N$32: C14.2, R20.1, R21.2
- removed net N$33: C15.1, IC6.5, R21.1
- removed net N$34: IC4.2
- removed net N$35: C14.1, IC6.6, IC6.7, R17.2
- removed net N$36: R22.1, R5.2
- removed net N$37: IC4.3
- removed net N$38: R24.1, R25.2
- removed net N$39: C16.1, R23.2, R25.1, R26.2
- removed net N$40: IC6.3, R26.1
- removed net N$41: IC6.1, R18.1
- removed net N$42: IC7.1, RG2.2
- removed net N$43: IC7.8, RG2.1
- removed net N$44: C17.1, IC7.6
- removed net N$45: C17.2, C18.1, R28.1
- removed net N$46: C18.2, IC8.5, R35.2
- removed net N$47: IC8.6, IC8.7, R28.2, R29.2
- removed net N$48: C19.2, R29.1, R30.2
- removed net N$49: C20.1, IC8.3, R30.1
- removed net N$50: C19.1, IC8.1, IC8.2, R33.2
- removed net N$51: IC9.2, R31.1, R32.2
- removed net N$52: C21.2, R33.1, R34.2
- removed net N$53: C22.1, IC9.5, R34.1
- removed net N$54: IC7.2
- removed net N$55: C21.1, IC9.6, IC9.7, R31.2
- removed net N$56: R27.2, R35.1
- removed net N$57: IC7.3
- removed net N$58: R37.1, R38.2
- removed net N$59: C23.1, R36.2, R38.1, R39.2
- removed net N$60: IC9.3, R39.1
- removed net N$61: IC10.1, RG3.2
- removed net N$62: IC10.8, RG3.1
- removed net N$63: C24.1, IC10.6
- removed net N$64: C24.2, C25.1, R41.1
- removed net N$65: C25.2, IC11.5, R48.2
- removed net N$66: IC11.6, IC11.7, R41.2, R42.2
- removed net N$67: C26.2, R42.1, R43.2
- removed net N$68: C27.1, IC11.3, R43.1
- removed net N$69: C26.1, IC11.1, IC11.2, R46.2
- removed net N$70: IC12.2, R44.1, R45.2
- removed net N$71: C28.2, R46.1, R47.2
- removed net N$72: C29.1, IC12.5, R47.1
- removed net N$73: IC10.2
- removed net N$74: C28.1, IC12.6, IC12.7, R44.2
- removed net N$75: R40.2, R48.1
- removed net N$76: IC10.3
- removed net N$77: R50.1, R51.2
- removed net N$78: C30.1, R49.2, R51.1, R52.2
- removed net N$79: IC12.3, R52.1
- removed net N$80: IC12.1, R45.1
- removed net N$81: IC9.1, R32.1
- net +9V: no longer IC10.7, IC11.8, IC12.8, IC4.7, IC5.8, IC6.8, IC7.7, IC8.8, IC9.8, R23.1, R36.1, R49.1
- net -9V: no longer IC10.4, IC11.4, IC12.4, IC4.4, IC5.4, IC6.4, IC7.4, IC8.4, IC9.4, R24.2, R37.2, R50.2
- net 0: now also J1.SLEEVE; no longer C13.2, C15.2, C16.2, C20.2, C22.2, C23.2, C27.2, C29.2, C30.2, IC10.5, IC4.5, IC7.5, R27.1, R40.1, R5.1
- net N$15: now also R5.1; no longer R11.2
- net N$16: now also C6.1, R14.2, R5.2; no longer IC4.1, RG1.2
- net N$20: now also R5.3; no longer C6.1, R11.1, R14.2
- net N$26: now also J1.TSH
- net N$3: now also J1.RING
