File: schematics/hand sensor/EMG3.sch (EAGLE design)
At the start: 100 parts, among them IC1 INA118P, IC10 INA118P, IC11 OP275P, IC12 OP275P, IC2 OP275P, IC3 OP275P, IC4 INA118P, IC5 OP275P, IC6 OP275P, IC7 INA118P, IC8 OP275P, IC9 OP275P

Commit message: implement NN, dummy data, 3d hand
Parts:
- removed C10, C11, C17, C18, C24, C25: 220nF, rcl:C-EU050-035X075
- removed C12, C19, C26: 33nF, rcl:C-EU050-035X075
- removed C13, C20, C27: 22nF, rcl:C-EU050-035X075
- removed C14, C21, C28: 100nF, rcl:C-EU050-035X075
- removed C15, C16, C22, C23, C29, C30: 10nF, rcl:C-EU050-035X075
- removed IC10, IC4, IC7: INA118P, burr-brown:INA118P
- removed IC11, IC12, IC5, IC6, IC8, IC9: OP275P, linear:OP275P
- removed R11, R25, R38, R51: 200, rcl:R-US_0207/7
- removed R15, R29, R42: 6.8k, rcl:R-US_0207/7
- removed R16, R21, R30, R34, R43, R47: 20k, rcl:R-US_0207/7
- removed R17, R26, R31, R39, R44, R52, RG1, RG2, RG3: 1K, rcl:R-US_0207/7
- removed R18, R32, R45: 100K, rcl:R-US_0207/7
- removed R20, R33, R46: 5.1k, rcl:R-US_0207/7
- removed R22, R27, R35, R40, R48: 51k, rcl:R-US_0207/7
- removed R23, R24, R36, R37, R49, R50: 10k, rcl:R-US_0207/7
- removed R28, R41, R9: 51K, rcl:R-US_0207/7
- added J1: AUDIO_JACK_3.5MM_PTH, SparkFun-Connectors:AUDIO_JACK_3.5MM_PTH
- C1, C2, C3, C4, C8, C9: device rcl:C-EU050-035X075 -> rcl:C-EU050-025X075
- R1, R10, R12, R13, R14, R19, R2, R3, R4, R6, R7, R8, RG: device rcl:R-US_0207/7 -> rcl:R-US_0207/12
- R5: value 51k -> (none); device rcl:R-US_0207/7 -> rcl:R-TRIMM64W
Connections:
- removed net N$18 (its old number): IC4.RG@1, RG1.1
- removed net N$21: C10.1, IC4.OUT
- removed net N$22: C10.2, C11.1, R9.1
- removed net N$24: C11.2, IC5B.+IN, R22.2
- removed net N$27: IC5B.-IN, IC5B.OUT, R15.2, R9.2
- removed net N$28: C12.2, R15.1, R16.2
- removed net N$29: C13.1, IC5A.+IN, R16.1
- removed net N$30: C12.1, IC5A.-IN, IC5A.OUT, R20.2
- removed net N$31: IC6A.-IN, R17.1, R18.2
- removed net N$32: C14.2, R20.1, R21.2
- removed net N$33: C15.1, IC6B.+IN, R21.1
- removed net N$34: IC4.-IN
- removed net N$35: C14.1, IC6B.-IN, IC6B.OUT, R17.2
- removed net N$36: R22.1, R5.2
- removed net N$37: IC4.+IN
- removed net N$38: R24.1, R25.2
- removed net N$39: C16.1, R23.2, R25.1, R26.2
- removed net N$40: IC6A.+IN, R26.1
- removed net N$41: IC6A.OUT, R18.1
- removed net N$42: IC7.RG, RG2.2
- removed net N$43: IC7.RG@1, RG2.1
- removed net N$44: C17.1, IC7.OUT
- removed net N$45: C17.2, C18.1, R28.1
- removed net N$46: C18.2, IC8B.+IN, R35.2
- removed net N$47: IC8B.-IN, IC8B.OUT, R28.2, R29.2
- removed net N$48: C19.2, R29.1, R30.2
- removed net N$49: C20.1, IC8A.+IN, R30.1
- removed net N$50: C19.1, IC8A.-IN, IC8A.OUT, R33.2
- removed net N$51: IC9A.-IN, R31.1, R32.2
- removed net N$52: C21.2, R33.1, R34.2
- removed net N$53: C22.1, IC9B.+IN, R34.1
- removed net N$54: IC7.-IN
- removed net N$55: C21.1, IC9B.-IN, IC9B.OUT, R31.2
- removed net N$56: R27.2, R35.1
- removed net N$57: IC7.+IN
- removed net N$58: R37.1, R38.2
- removed net N$59: C23.1, R36.2, R38.1, R39.2
- removed net N$60: IC9A.+IN, R39.1
- removed net N$61: IC10.RG, RG3.2
- removed net N$62: IC10.RG@1, RG3.1
- removed net N$63: C24.1, IC10.OUT
- removed net N$64: C24.2, C25.1, R41.1
- removed net N$65: C25.2, IC11B.+IN, R48.2
- removed net N$66: IC11B.-IN, IC11B.OUT, R41.2, R42.2
- removed net N$67: C26.2, R42.1, R43.2
- removed net N$68: C27.1, IC11A.+IN, R43.1
- removed net N$69: C26.1, IC11A.-IN, IC11A.OUT, R46.2
- removed net N$70: IC12A.-IN, R44.1, R45.2
- removed net N$71: C28.2, R46.1, R47.2
- removed net N$72: C29.1, IC12B.+IN, R47.1
- removed net N$73: IC10.-IN
- removed net N$74: C28.1, IC12B.-IN, IC12B.OUT, R44.2
- removed net N$75: R40.2, R48.1
- removed net N$76: IC10.+IN
- removed net N$77: R50.1, R51.2
- removed net N$78: C30.1, R49.2, R51.1, R52.2
- removed net N$79: IC12A.+IN, R52.1
- removed net N$80: IC12A.OUT, R45.1
- removed net N$81: IC9A.OUT, R32.1
- net +9V: now also R1.2, R2.2, R3.2, R4.2; no longer IC10.V+, IC11P.V+, IC12P.V+, IC4.V+, IC5P.V+, IC6P.V+, IC7.V+, IC8P.V+, IC9P.V+, R23.1, R36.1, R49.1
- net -9V: no longer IC10.V-, IC11P.V-, IC12P.V-, IC4.V-, IC5P.V-, IC6P.V-, IC7.V-, IC8P.V-, IC9P.V-, R24.2, R37.2, R50.2
- net 0: now also J1.SLEEVE; no longer C13.2, C15.2, C16.2, C20.2, C22.2, C23.2, C27.2, C29.2, C30.2, IC10.REF, IC4.REF, IC7.REF, R27.1, R40.1, R5.1
- net N$1: now also R1.1
- net N$15: now also R5.A; no longer R11.2
- net N$16: now also C6.1, R14.2, R5.S; no longer IC4.RG, RG1.2
- net N$2: now also R2.1
- net N$20: now also R5.E; no longer C6.1, R11.1, R14.2
- net N$26: now also J1.TSH
- net N$3: now also J1.RING, R3.1
- net N$4: now also R4.1
Other:
- moved on the sheet: C6, R10, R14, R7, R8
