File: schematics/hand sensor/IRcircuit.sch (EAGLE design)
At the start: 19 parts, among them IC1 AD712N, IC2 AD712N, T1 BPX81, T2 BPX81, T3 BPX81, T4 BPX81, U1 ULN2803ADWR

Commit message: implement NN, dummy data, 3d hand
Parts:
- removed D1, D2, D3, D4: SFH482, led:SFH482
- removed R1, R3, R4: 150, ngspice-simulation:R
- removed R5, R6, R7, R8: (no value), ngspice-simulation:R
- removed T1, T2, T3, T4: BPX81, opto-trans-siemens:BPX81
- removed U1: ULN2803ADWR, imported:ULN2803ADWR
- added C1, C2: 1uF, rcl:C-EU050-025X075
- added ICSP: ICSP, SmartPrj:PINHD-2X3
- added J2, J3: 8x1F-H8.5, SmartPrj:PINHD-1X8
- added J4: 6x1F-H8.5, SmartPrj:PINHD-1X6
- added JP1: 10x1F-H8.5, SmartPrj:PINHD-1X10
- added NIR1, NIR2, NIR3, NIR4: (no value), con-lstb:MA04-1
- added POT1, POT2, POT3, POT4, POT5, POT6, POT7, POT8: (no value), con-lstb:MA03-1
- added R53, R54, R55, R60: 68, rcl:R-US_0207/12
- added R56, R62, R63, R64: 10k, rcl:R-US_0207/12
- added U2: ULN2803AN, transistor-arrays:ULN2803AN
- added X1, X2, X3, X4: 332-02, con-garry:332-02
- IC1, IC2: value AD712N -> MCP3208c; device analog-devices:AD712N -> ic-package:DIL16
- R2: value 150 -> 10k; device ngspice-simulation:R -> rcl:R-TRIMMT93YA
Connections:
- removed net +9V: R1.2, R2.2, R3.2, R4.2, T1.C, T2.C, T3.C, T4.C, U1.COM
- removed net N$1: D1.A, R1.1
- removed net N$2: D2.A, R2.1
- removed net N$3: D3.A, R3.1
- removed net N$4: D4.A, R4.1
- removed net N$5: D1.C, U1.1C
- removed net SIG1: R5.2, T1.E
- removed net SIG2: R6.2, T2.E
- removed net SIG3: R7.2, T3.E
- removed net SIG4: R8.2, T4.E
- new net +5V: C1.2, C2.2, IC1.16, IC2.15, IC2.16, ICSP.2, J3.5, NIR1.4, NIR2.4, NIR3.4, NIR4.4, POT1.3, POT2.3, POT3.3, POT4.3, POT5.3, POT6.3, POT7.3, POT8.3, R2.A, R53.2, R54.2, R55.2, R60.2, U2.COM
- new net CLK: IC1.13, IC2.13, ICSP.3
- new net CS1: IC1.10, JP1.3
- new net CS2: IC2.10, JP1.4
- new net DGND: IC1.9, IC2.9, ICSP.6, J3.6, J3.7, JP1.7
- new net DIN: IC1.11, IC2.11, ICSP.4
- new net DOUT: IC1.12, IC2.12, ICSP.1
- new net EMG1: IC1.1, X1-1.S
- new net EMG2: IC1.2, X2-1.S
- new net EMG3: IC1.3, X3-1.S
- new net EMG4: IC1.4, X4-1.S
- new net N$100: NIR3.1, R53.1
- new net N$101: NIR4.1, R60.1
- new net N$12: IC2.5, POT5.2
- new net N$13: IC2.7, POT7.2
- new net N$14: IC2.8, POT8.2
- new net N$18: ICSP.5
- new net N$20: IC1.15, R2.S
- new net N$21: NIR1.2, U2.1C
- new net N$22: NIR2.2, U2.3C
- new net N$23: NIR3.2, U2.5C
- new net N$24: NIR4.2, U2.7C
- new net N$26: JP1.6
- new net N$6: IC2.6, POT6.2
- new net N$7: IC2.1, POT1.2
- new net N$98: NIR1.1, R55.1
- new net N$99: NIR2.1, R54.1
- new net NIR1: IC1.5, NIR1.3, R64.2
- new net NIR2: IC1.6, NIR2.3, R63.2
- new net NIR3: IC1.7, NIR3.3, R62.2
- new net NIR4: IC1.8, NIR4.3, R56.2
- net 0: now also C1.1, C2.1, IC1.14, IC2.14, POT1.1, POT2.1, POT3.1, POT4.1, POT5.1, POT6.1, POT7.1, POT8.1, R2.E, R56.1, R62.1, R63.1, R64.1, U2.2B, U2.4B, U2.6B, U2.8B, U2.GND; no longer R5.1, R6.1, R7.1, R8.1, U1.GND
- net ARDUINO1: now also J2.3, U2.1B; no longer U1.1B
- net ARDUINO2: now also J2.5, U2.3B; no longer U1.3B
- net ARDUINO3: now also J2.6, U2.5B; no longer U1.5B
- net ARDUINO4: now also JP1.2, U2.7B; no longer U1.7B
- net N$10: now also IC2.3, POT3.2; no longer D3.C, U1.5C
- net N$11: now also IC2.4, POT4.2; no longer D4.C, U1.7C
- net N$9: now also IC2.2, POT2.2; no longer D2.C, U1.3C
